Commit message: 2021年 04月 09日 星期五 11:05:51 CST

File: ur3_description/urdf/accessories.urdf.xacro (robot description, xacro)
@@ -1,6 +1,9 @@
 <?xml version="1.0"?>
 <robot xmlns:xacro="http://ros.org/wiki/xacro">
+  <!-- ur3 -->
   <xacro:include filename="$(find ur_description)/urdf/ur3.urdf.xacro" />
-<!-- Spawn arm -->
+  <!-- robotiq -->
+  <xacro:include filename="$(find robotiq_ft_sensor)/urdf/robotiq_ft300.urdf.xacro" />
+  <!-- Spawn arm -->
   <xacro:arg name="transmission_hw_interface" default="hardware_interface/PositionJointInterface"/>
   <xacro:arg name="kinematics_config" default="$(find ur_description)/config/ur3_default.yaml"/>
@@ -12,24 +15,9 @@
 	<parent link="mid_mount" />
 	<child link="ur3_arm_base_link" />
-	<origin xyz="0 0.0 0.0" rpy="0.0 0.0 -1.5708" />
+	<origin xyz="0 0.0 0.0" rpy="0.0 0.0 0.0" />
   </joint>
-  <!-- Sensor Mount and other custom parts -->
-  <link name="FT300_link">
-		<visual>
-			<geometry>
-				<cylinder length="0.04" radius="0.035"/>
-			</geometry>
-			<material name="black"/>
-		</visual>
-		<collision>
-			<geometry>
-				<cylinder length="0.04" radius="0.035"/>
-			</geometry>
-		</collision>
-   </link>
-  <joint name="FT300_joint" type="fixed">
-	  <origin xyz="0.02 0 0" rpy="0 1.57 0" />
-	  <parent link="ur3_arm_ee_link" />
-	  <child link="FT300_link" />
-  </joint>
+  <!-- robotiq -->
+  <xacro:robotiq_ft300 prefix="" parent="ur3_arm_ee_link" >
+    <origin xyz="-0.004 0 0" rpy="0 ${pi/2} 0 "/>
+  </xacro:robotiq_ft300>
 </robot>

File: ur3_description/urdf/ur3_ft300.urdf.xacro (robot description, xacro)
@@ -1,6 +1,5 @@
 <?xml version="1.0"?>
 <robot name="ur3" xmlns:xacro="http://ros.org/wiki/xacro">
-  <xacro:property name="PI" value="3.1415926535897931" />
-  <xacro:property name="connector_height" value="0.020" />
+  <xacro:property name="connector_height" value="0.0" />
   <material name="dark_grey"><color rgba="0.2 0.2 0.2 1.0" /></material>
   <material name="light_grey"><color rgba="0.4 0.4 0.4 1.0" /></material>
